Commit message: Updated URDF

File: ros2/src/bebopv2_description/urdf/bebopv2.xacro (robot description, xacro)
@@ -6,7 +6,7 @@
 <link name="base_link">
   <inertial>
-    <origin xyz="0.007385904694151062 -0.0004782319133016371 0.03368322966647506" rpy="0 0 0"/>
-    <mass value="2.683107573914711"/>
-    <inertia ixx="0.035466" iyy="0.017273" izz="0.025862" ixy="4.2e-05" iyz="-1.7e-05" ixz="-0.001118"/>
+    <origin xyz="-8.495725208879161e-05 0.002060204806872657 0.06042048201634313" rpy="0 0 0"/>
+    <mass value="10.498536136255769"/>
+    <inertia ixx="0.135473" iyy="0.076749" izz="0.084177" ixy="0.000202" iyz="-0.001328" ixz="-0.002579"/>
   </inertial>
   <visual>
@@ -24,219 +24,219 @@
   </collision>
 </link>
-<link name="hip_abduction_left_1_1">
-  <inertial>
-    <origin xyz="-0.0003217598941065208 0.06711052569446321 1.0147989649067783e-05" rpy="0 0 0"/>
-    <mass value="0.38495857785704823"/>
-    <inertia ixx="0.000878" iyy="0.000645" izz="0.000696" ixy="0.0" iyz="0.0" ixz="1e-06"/>
-  </inertial>
-  <visual>
-    <origin xyz="0.000262 -0.15 -0.000132" rpy="0 0 0"/>
-    <geometry>
-      <mesh filename="file://$(find bebopv2_description)/meshes/hip_abduction_left_1_1.stl" scale="0.001 0.001 0.001"/>
-    </geometry>
-    <material name="silver"/>
-  </visual>
-  <collision>
-    <origin xyz="0.000262 -0.15 -0.000132" rpy="0 0 0"/>
-    <geometry>
-      <mesh filename="file://$(find bebopv2_description)/meshes/hip_abduction_left_1_1.stl" scale="0.001 0.001 0.001"/>
-    </geometry>
-  </collision>
-</link>
-<link name="hip_abduction_right_1_1">
-  <inertial>
-    <origin xyz="-0.0003217940431635766 -0.06711052938146245 -1.023141995292347e-05" rpy="0 0 0"/>
-    <mass value="0.3849585610474383"/>
-    <inertia ixx="0.000878" iyy="0.000645" izz="0.000696" ixy="-0.0" iyz="0.0" ixz="-1e-06"/>
-  </inertial>
-  <visual>
-    <origin xyz="0.0 0.151 -0.0" rpy="0 0 0"/>
-    <geometry>
-      <mesh filename="file://$(find bebopv2_description)/meshes/hip_abduction_right_1_1.stl" scale="0.001 0.001 0.001"/>
-    </geometry>
-    <material name="silver"/>
-  </visual>
-  <collision>
-    <origin xyz="0.0 0.151 -0.0" rpy="0 0 0"/>
-    <geometry>
-      <mesh filename="file://$(find bebopv2_description)/meshes/hip_abduction_right_1_1.stl" scale="0.001 0.001 0.001"/>
-    </geometry>
-  </collision>
-</link>
-<link name="femur_left_1_1">
-  <inertial>
-    <origin xyz="0.03177134523380352 0.00031797747528269915 -0.18130160282671445" rpy="0 0 0"/>
-    <mass value="6.100588872036469"/>
-    <inertia ixx="0.082959" iyy="0.08488" izz="0.005962" ixy="-8e-06" iyz="0.000373" ixz="0.005077"/>
-  </inertial>
-  <visual>
-    <origin xyz="-0.029288 -0.22 -0.000132" rpy="0 0 0"/>
-    <geometry>
-      <mesh filename="file://$(find bebopv2_description)/meshes/femur_left_1_1.stl" scale="0.001 0.001 0.001"/>
-    </geometry>
-    <material name="silver"/>
-  </visual>
-  <collision>
-    <origin xyz="-0.029288 -0.22 -0.000132" rpy="0 0 0"/>
-    <geometry>
-      <mesh filename="file://$(find bebopv2_description)/meshes/femur_left_1_1.stl" scale="0.001 0.001 0.001"/>
-    </geometry>
-  </collision>
-</link>
-<link name="femur_right_1_1">
-  <inertial>
-    <origin xyz="0.0321027922345207 -0.00031797682024858887 -0.18130148887841674" rpy="0 0 0"/>
-    <mass value="6.100585251669615"/>
-    <inertia ixx="0.082959" iyy="0.084903" izz="0.005985" ixy="1.4e-05" iyz="-0.000373" ixz="0.005232"/>
-  </inertial>
-  <visual>
-    <origin xyz="-0.02955 0.221 0.0" rpy="0 0 0"/>
-    <geometry>
-      <mesh filename="file://$(find bebopv2_description)/meshes/femur_right_1_1.stl" scale="0.001 0.001 0.001"/>
-    </geometry>
-    <material name="silver"/>
-  </visual>
-  <collision>
-    <origin xyz="-0.02955 0.221 0.0" rpy="0 0 0"/>
-    <geometry>
-      <mesh filename="file://$(find bebopv2_description)/meshes/femur_right_1_1.stl" scale="0.001 0.001 0.001"/>
-    </geometry>
-  </collision>
-</link>
-<link name="shin_left_1_1">
-  <inertial>
-    <origin xyz="3.887590066825597e-05 0.016598133015893995 -0.12318420193029112" rpy="0 0 0"/>
-    <mass value="0.23016891060875985"/>
-    <inertia ixx="0.001921" iyy="0.001941" izz="4.3e-05" ixy="-0.0" iyz="-1.2e-05" ixz="-0.0"/>
-  </inertial>
-  <visual>
-    <origin xyz="-0.066788 -0.2477 0.293902" rpy="0 0 0"/>
-    <geometry>
-      <mesh filename="file://$(find bebopv2_description)/meshes/shin_left_1_1.stl" scale="0.001 0.001 0.001"/>
-    </geometry>
-    <material name="silver"/>
-  </visual>
-  <collision>
-    <origin xyz="-0.066788 -0.2477 0.293902" rpy="0 0 0"/>
-    <geometry>
-      <mesh filename="file://$(find bebopv2_description)/meshes/shin_left_1_1.stl" scale="0.001 0.001 0.001"/>
-    </geometry>
-  </collision>
-</link>
-<link name="shin_right_1_1">
-  <inertial>
-    <origin xyz="-0.0021886908544472145 -0.016598132485373535 -0.12316472976088472" rpy="0 0 0"/>
-    <mass value="0.23016883140801822"/>
-    <inertia ixx="0.001921" iyy="0.001941" izz="4.4e-05" ixy="0.0" iyz="1.2e-05" ixz="-3.2e-05"/>
-  </inertial>
-  <visual>
-    <origin xyz="-0.06705 0.2487 0.294034" rpy="0 0 0"/>
-    <geometry>
-      <mesh filename="file://$(find bebopv2_description)/meshes/shin_right_1_1.stl" scale="0.001 0.001 0.001"/>
-    </geometry>
-    <material name="silver"/>
-  </visual>
-  <collision>
-    <origin xyz="-0.06705 0.2487 0.294034" rpy="0 0 0"/>
-    <geometry>
-      <mesh filename="file://$(find bebopv2_description)/meshes/shin_right_1_1.stl" scale="0.001 0.001 0.001"/>
-    </geometry>
-  </collision>
-</link>
-<link name="foot_left_1_1">
-  <inertial>
-    <origin xyz="0.02219188787582449 -0.016069983036660074 -0.040821402975144694" rpy="0 0 0"/>
-    <mass value="0.938066903777968"/>
-    <inertia ixx="0.001351" iyy="0.003336" izz="0.003073" ixy="-9.6e-05" iyz="0.00018" ixz="0.000268"/>
-  </inertial>
-  <visual>
-    <origin xyz="-0.066793 -0.2477 0.547402" rpy="0 0 0"/>
-    <geometry>
-      <mesh filename="file://$(find bebopv2_description)/meshes/foot_left_1_1.stl" scale="0.001 0.001 0.001"/>
-    </geometry>
-    <material name="silver"/>
-  </visual>
-  <collision>
-    <origin xyz="-0.066793 -0.2477 0.547402" rpy="0 0 0"/>
-    <geometry>
-      <mesh filename="file://$(find bebopv2_description)/meshes/foot_left_1_1.stl" scale="0.001 0.001 0.001"/>
-    </geometry>
-  </collision>
-</link>
-<link name="foot_right_1_1">
-  <inertial>
-    <origin xyz="0.02218978231016064 0.016069982543298805 -0.040816882308905234" rpy="0 0 0"/>
-    <mass value="0.9380669235063296"/>
-    <inertia ixx="0.001352" iyy="0.003336" izz="0.003073" ixy="9.6e-05" iyz="-0.000181" ixz="0.000268"/>
-  </inertial>
-  <visual>
-    <origin xyz="-0.062621 0.2487 0.547495" rpy="0 0 0"/>
-    <geometry>
-      <mesh filename="file://$(find bebopv2_description)/meshes/foot_right_1_1.stl" scale="0.001 0.001 0.001"/>
-    </geometry>
-    <material name="silver"/>
-  </visual>
-  <collision>
-    <origin xyz="-0.062621 0.2487 0.547495" rpy="0 0 0"/>
-    <geometry>
-      <mesh filename="file://$(find bebopv2_description)/meshes/foot_right_1_1.stl" scale="0.001 0.001 0.001"/>
-    </geometry>
-  </collision>
-</link>
+<link name="femur_left_1">
+  <inertial>
+    <origin xyz="0.03177093685295705 0.0003179774752826714 -0.18130160282671148" rpy="0 0 0"/>
+    <mass value="1.741996667034525"/>
+    <inertia ixx="0.023689" iyy="0.024237" izz="0.001703" ixy="-2e-06" iyz="0.000107" ixz="0.00145"/>
+  </inertial>
+  <visual>
+    <origin xyz="-0.025761 -0.2205 -0.013132" rpy="0 0 0"/>
+    <geometry>
+      <mesh filename="file://$(find bebopv2_description)/meshes/femur_left_1.stl" scale="0.001 0.001 0.001"/>
+    </geometry>
+    <material name="silver"/>
+  </visual>
+  <collision>
+    <origin xyz="-0.025761 -0.2205 -0.013132" rpy="0 0 0"/>
+    <geometry>
+      <mesh filename="file://$(find bebopv2_description)/meshes/femur_left_1.stl" scale="0.001 0.001 0.001"/>
+    </geometry>
+  </collision>
+</link>
+<link name="femur_right_1">
+  <inertial>
+    <origin xyz="0.03210238385367442 -0.00031797682024858887 -0.18130148887841402" rpy="0 0 0"/>
+    <mass value="1.741992832749943"/>
+    <inertia ixx="0.023688" iyy="0.024244" izz="0.001709" ixy="4e-06" iyz="-0.000107" ixz="0.001494"/>
+  </inertial>
+  <visual>
+    <origin xyz="-0.026023 0.2195 -0.013" rpy="0 0 0"/>
+    <geometry>
+      <mesh filename="file://$(find bebopv2_description)/meshes/femur_right_1.stl" scale="0.001 0.001 0.001"/>
+    </geometry>
+    <material name="silver"/>
+  </visual>
+  <collision>
+    <origin xyz="-0.026023 0.2195 -0.013" rpy="0 0 0"/>
+    <geometry>
+      <mesh filename="file://$(find bebopv2_description)/meshes/femur_right_1.stl" scale="0.001 0.001 0.001"/>
+    </geometry>
+  </collision>
+</link>
+<link name="shin_left_1">
+  <inertial>
+    <origin xyz="3.846626426318167e-05 0.01659813777561367 -0.12318432363895004" rpy="0 0 0"/>
+    <mass value="0.11370113593752607"/>
+    <inertia ixx="0.000949" iyy="0.000959" izz="2.1e-05" ixy="-0.0" iyz="-6e-06" ixz="-0.0"/>
+  </inertial>
+  <visual>
+    <origin xyz="-0.063261 -0.2482 0.280902" rpy="0 0 0"/>
+    <geometry>
+      <mesh filename="file://$(find bebopv2_description)/meshes/shin_left_1.stl" scale="0.001 0.001 0.001"/>
+    </geometry>
+    <material name="silver"/>
+  </visual>
+  <collision>
+    <origin xyz="-0.063261 -0.2482 0.280902" rpy="0 0 0"/>
+    <geometry>
+      <mesh filename="file://$(find bebopv2_description)/meshes/shin_left_1.stl" scale="0.001 0.001 0.001"/>
+    </geometry>
+  </collision>
+</link>
+<link name="shin_right_1">
+  <inertial>
+    <origin xyz="-0.0021891088643529594 -0.016598079567325258 -0.12316565094474391" rpy="0 0 0"/>
+    <mass value="0.11369998148988655"/>
+    <inertia ixx="0.000949" iyy="0.000959" izz="2.2e-05" ixy="0.0" iyz="6e-06" ixz="-1.6e-05"/>
+  </inertial>
+  <visual>
+    <origin xyz="-0.063523 0.2472 0.281034" rpy="0 0 0"/>
+    <geometry>
+      <mesh filename="file://$(find bebopv2_description)/meshes/shin_right_1.stl" scale="0.001 0.001 0.001"/>
+    </geometry>
+    <material name="silver"/>
+  </visual>
+  <collision>
+    <origin xyz="-0.063523 0.2472 0.281034" rpy="0 0 0"/>
+    <geometry>
+      <mesh filename="file://$(find bebopv2_description)/meshes/shin_right_1.stl" scale="0.001 0.001 0.001"/>
+    </geometry>
+  </collision>
+</link>
+<link name="foot_left_1">
+  <inertial>
+    <origin xyz="0.022192420913894034 -0.01606998038885915 -0.0408213906831868" rpy="0 0 0"/>
+    <mass value="0.6420025158679283"/>
+    <inertia ixx="0.000925" iyy="0.002283" izz="0.002103" ixy="-6.5e-05" iyz="0.000124" ixz="0.000184"/>
+  </inertial>
+  <visual>
+    <origin xyz="-0.063265 -0.2482 0.534402" rpy="0 0 0"/>
+    <geometry>
+      <mesh filename="file://$(find bebopv2_description)/meshes/foot_left_1.stl" scale="0.001 0.001 0.001"/>
+    </geometry>
+    <material name="silver"/>
+  </visual>
+  <collision>
+    <origin xyz="-0.063265 -0.2482 0.534402" rpy="0 0 0"/>
+    <geometry>
+      <mesh filename="file://$(find bebopv2_description)/meshes/foot_left_1.stl" scale="0.001 0.001 0.001"/>
+    </geometry>
+  </collision>
+</link>
+<link name="foot_right_1">
+  <inertial>
+    <origin xyz="0.02218934865992219 0.016069987053803497 -0.04081687775985443" rpy="0 0 0"/>
+    <mass value="0.6420010099946694"/>
+    <inertia ixx="0.000925" iyy="0.002283" izz="0.002103" ixy="6.5e-05" iyz="-0.000124" ixz="0.000184"/>
+  </inertial>
+  <visual>
+    <origin xyz="-0.059094 0.2472 0.534495" rpy="0 0 0"/>
+    <geometry>
+      <mesh filename="file://$(find bebopv2_description)/meshes/foot_right_1.stl" scale="0.001 0.001 0.001"/>
+    </geometry>
+    <material name="silver"/>
+  </visual>
+  <collision>
+    <origin xyz="-0.059094 0.2472 0.534495" rpy="0 0 0"/>
+    <geometry>
+      <mesh filename="file://$(find bebopv2_description)/meshes/foot_right_1.stl" scale="0.001 0.001 0.001"/>
+    </geometry>
+  </collision>
+</link>
+<link name="hip_abduction_right_1">
+  <inertial>
+    <origin xyz="-0.0003222024240098673 -0.06711052938146264 -1.0231419950193846e-05" rpy="0 0 0"/>
+    <mass value="1.000019792580193"/>
+    <inertia ixx="0.002281" iyy="0.001675" izz="0.001808" ixy="-1e-06" iyz="0.0" ixz="-2e-06"/>
+  </inertial>
+  <visual>
+    <origin xyz="0.003527 0.1495 -0.013" rpy="0 0 0"/>
+    <geometry>
+      <mesh filename="file://$(find bebopv2_description)/meshes/hip_abduction_right_1.stl" scale="0.001 0.001 0.001"/>
+    </geometry>
+    <material name="silver"/>
+  </visual>
+  <collision>
+    <origin xyz="0.003527 0.1495 -0.013" rpy="0 0 0"/>
+    <geometry>
+      <mesh filename="file://$(find bebopv2_description)/meshes/hip_abduction_right_1.stl" scale="0.001 0.001 0.001"/>
+    </geometry>
+  </collision>
+</link>
+<link name="hip_abduction_left_1">
+  <inertial>
+    <origin xyz="-0.0003221682749529886 0.0671105256944631 1.0147989652034214e-05" rpy="0 0 0"/>
+    <mass value="1.0000098137346085"/>
+    <inertia ixx="0.002281" iyy="0.001675" izz="0.001808" ixy="1e-06" iyz="0.0" ixz="2e-06"/>
+  </inertial>
+  <visual>
+    <origin xyz="0.003789 -0.1505 -0.013132" rpy="0 0 0"/>
+    <geometry>
+      <mesh filename="file://$(find bebopv2_description)/meshes/hip_abduction_left_1.stl" scale="0.001 0.001 0.001"/>
+    </geometry>
+    <material name="silver"/>
+  </visual>
+  <collision>
+    <origin xyz="0.003789 -0.1505 -0.013132" rpy="0 0 0"/>
+    <geometry>
+      <mesh filename="file://$(find bebopv2_description)/meshes/hip_abduction_left_1.stl" scale="0.001 0.001 0.001"/>
+    </geometry>
+  </collision>
+</link>
+<joint name="femur_left_joint" type="revolute">
+  <origin xyz="0.02955 0.07 0.0" rpy="0 0 0"/>
+  <parent link="hip_abduction_left_1"/>
+  <child link="femur_left_1"/>
+  <axis xyz="1.0 -0.0 0.0"/>
+  <limit upper="0.785398" lower="-0.349066" effort="100" velocity="100"/>
+</joint>
+<joint name="femur_right_joint" type="revolute">
+  <origin xyz="0.02955 -0.07 0.0" rpy="0 0 0"/>
+  <parent link="hip_abduction_right_1"/>
+  <child link="femur_right_1"/>
+  <axis xyz="1.0 -0.0 -0.0"/>
+  <limit upper="0.349066" lower="-0.785398" effort="100" velocity="100"/>
+</joint>
+<joint name="shin_left_joint" type="revolute">
+  <origin xyz="0.0375 0.0277 -0.294034" rpy="0 0 0"/>
+  <parent link="femur_left_1"/>
+  <child link="shin_left_1"/>
+  <axis xyz="0.0 1.0 0.0"/>
+  <limit upper="1.570796" lower="-0.785398" effort="100" velocity="100"/>
+</joint>
+<joint name="shin_right_joint" type="revolute">
+  <origin xyz="0.0375 -0.0277 -0.294034" rpy="0 0 0"/>
+  <parent link="femur_right_1"/>
+  <child link="shin_right_1"/>
+  <axis xyz="-0.0 -1.0 -0.0"/>
+  <limit upper="0.785398" lower="-1.570796" effort="100" velocity="100"/>
+</joint>
+<joint name="foot_left_joint" type="revolute">
+  <origin xyz="4e-06 0.0 -0.2535" rpy="0 0 0"/>
+  <parent link="shin_left_1"/>
+  <child link="foot_left_1"/>
+  <axis xyz="-0.0 1.0 0.0"/>
+  <limit upper="0.523599" lower="-0.523599" effort="100" velocity="100"/>
+</joint>
+<joint name="foot_right_joint" type="revolute">
+  <origin xyz="-0.004429 0.0 -0.253461" rpy="0 0 0"/>
+  <parent link="shin_right_1"/>
+  <child link="foot_right_1"/>
+  <axis xyz="-0.0 -1.0 -0.0"/>
+  <limit upper="0.523599" lower="-0.523599" effort="100" velocity="100"/>
+</joint>
+<joint name="hip_abduction_right_joint" type="revolute">
+  <origin xyz="-0.003527 -0.1495 0.013" rpy="0 0 0"/>
+  <parent link="base_link"/>
+  <child link="hip_abduction_right_1"/>
+  <axis xyz="-0.0 -1.0 -0.0"/>
+  <limit upper="0.785398" lower="-0.785398" effort="100" velocity="100"/>
+</joint>
 <joint name="hip_abduction_left_joint" type="revolute">
-  <origin xyz="-0.000262 0.15 0.000132" rpy="0 0 0"/>
+  <origin xyz="-0.003789 0.1505 0.013132" rpy="0 0 0"/>
   <parent link="base_link"/>
-  <child link="hip_abduction_left_1_1"/>
+  <child link="hip_abduction_left_1"/>
   <axis xyz="0.0 1.0 -0.0"/>
   <limit upper="0.785398" lower="-0.785398" effort="100" velocity="100"/>
 </joint>
-<joint name="hip_abduction_right_joint" type="revolute">
-  <origin xyz="0.0 -0.151 0.0" rpy="0 0 0"/>
-  <parent link="base_link"/>
-  <child link="hip_abduction_right_1_1"/>
-  <axis xyz="-0.0 -1.0 0.0"/>
-  <limit upper="0.785398" lower="-0.785398" effort="100" velocity="100"/>
-</joint>
-<joint name="femur_left_joint" type="revolute">
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
Commit message: sim(bebop-v2): minimal standing experiment + 7kg torso mass correction Bench measurement showed the real torso is 7.0 kg, not the 10.5 kg the CAD-derived USD claimed. Combined with the kitchen-sink config's 2x mass scaling, the previous balance policy was trained on a ~21 kg torso -- 3x reality -- which is the most likely root cause of the robot standing in sim but not in real. Mass fix: - physics.usda: base_link mass 10.498536 -> 7.0, diagonalInertia   scaled by 7.0/10.498536 = 0.66676 (CoM unchanged, still   CAD-derived; needs a swing test before being trusted). - bebopv2.xacro: mirrored fix in the URDF inertia tensor for ROS   consistency. New Isaac-BebopV2-Standing-v0 task: a deliberately minimal "just stand" experiment, evolved in place from v0 through v0.5 with one knob added per iteration so each addition's effect is attributable: - v0:   alive + flat_orientation + base_height + joint_pos_limits         only; plain 8-dim JointPositionActionCfg; IMU + encoders         kept (no balance task without them). Policy stood but with         foot oscillation and horizontal drift. - v0.1: + action_rate_l2 (-0.05). Suppressed jitter. - v0.2: + foot_flat (1.0, std=0.15). Closed the heels-only         balance loophole the policy reward-hacked into. - v0.3: + Gaussian observation noise on the IMU + encoder obs         terms, magnitudes matched to the BNO085 / Robstride         hardware envelope. Exposed a small lateral rocking from         the fixed kp=40 hip abduction joints. - v0.4: switched action term to VariableImpedanceJointActionCfg         (24-dim raw -> 8 pos + 8 kp + 8 kd, firmware-compatible).         Policy raises hip-abduction kp during stance, rocking gone. - v0.5: tightened max_pos_step_per_tick on the position channel         from 1.0 (effectively unbounded) to 0.020 = 2 rad/s @         100 Hz. Matches the firmware safety target. Joint motion         is visibly smoother and flat_orientation / error_vel_yaw         actually improved -- the slew clamp forces forward planning         and beats reactive control for steady-state. Deployment lockstep: firmware/bebop-linux/config/bebop_v2.yaml defaults.slew.max_pos_step_per_tick is currently 0.015 and MUST be raised to 0.020 in lockstep before deploying this v0.5 checkpoint or the firmware will clip more tightly than sim. Knobs deferred for future iterations: action delay (action_delay_steps), IMU update-rate staleness (ImuCfg.update_period 0.0 -> 0.05), mass / friction / CoM domain randomization, actuator Coulomb friction, mid-episode pushes.

File: ros2/src/bebopv2_description/urdf/bebopv2.xacro (robot description, xacro)
@@ -6,7 +6,14 @@
 <link name="base_link">
   <inertial>
+    <!-- Mass + inertia adjusted from CAD value (10.4985 kg) to bench-measured
+         real torso (7.0 kg). Inertia tensor scaled by 7.0/10.4985 = 0.66676;
+         this assumes the geometric *distribution* of mass is unchanged and
+         only the total density dropped. The CoM is still CAD-derived and
+         needs a swing-test measurement before being trusted on the real
+         robot (battery + cables + electronics are not in the CAD model).
+         Keep this in sync with sim/usd/bebopv2/payloads/Physics/physics.usda. -->
     <origin xyz="-8.495725208879161e-05 0.002060204806872657 0.06042048201634313" rpy="0 0 0"/>
-    <mass value="10.498536136255769"/>
-    <inertia ixx="0.135473" iyy="0.076749" izz="0.084177" ixy="0.000202" iyz="-0.001328" ixz="-0.002579"/>
+    <mass value="7.0"/>
+    <inertia ixx="0.090323" iyy="0.051177" izz="0.056127" ixy="0.000135" iyz="-0.000885" ixz="-0.001719"/>
   </inertial>
   <visual>
