Commit message: exported new urdf with updated feet design

File: ros2/src/bebopv2_description/urdf/bebopv2.xacro (robot description, xacro)
@@ -64,44 +64,4 @@
   </collision>
 </link>
-<link name="foot_left_1">
-  <inertial>
-    <origin xyz="0.022192420913881364 -0.016069975495289518 -0.04082137886907555" rpy="0 0 0"/>
-    <mass value="0.6420025158679283"/>
-    <inertia ixx="0.000925" iyy="0.002283" izz="0.002103" ixy="-6.5e-05" iyz="0.000124" ixz="0.000184"/>
-  </inertial>
-  <visual>
-    <origin xyz="-0.063265 -0.1782 0.674402" rpy="0 0 0"/>
-    <geometry>
-      <mesh filename="file://$(find bebopv2_description)/meshes/foot_left_1.stl" scale="0.001 0.001 0.001"/>
-    </geometry>
-    <material name="silver"/>
-  </visual>
-  <collision>
-    <origin xyz="-0.063265 -0.1782 0.674402" rpy="0 0 0"/>
-    <geometry>
-      <mesh filename="file://$(find bebopv2_description)/meshes/foot_left_1.stl" scale="0.001 0.001 0.001"/>
-    </geometry>
-  </collision>
-</link>
-<link name="foot_right_1">
-  <inertial>
-    <origin xyz="0.022189348659933113 0.016069982160241636 -0.04081688957395602" rpy="0 0 0"/>
-    <mass value="0.6420010099946694"/>
-    <inertia ixx="0.000925" iyy="0.002283" izz="0.002103" ixy="6.5e-05" iyz="-0.000124" ixz="0.000184"/>
-  </inertial>
-  <visual>
-    <origin xyz="-0.059094 0.178 0.674495" rpy="0 0 0"/>
-    <geometry>
-      <mesh filename="file://$(find bebopv2_description)/meshes/foot_right_1.stl" scale="0.001 0.001 0.001"/>
-    </geometry>
-    <material name="silver"/>
-  </visual>
-  <collision>
-    <origin xyz="-0.059094 0.178 0.674495" rpy="0 0 0"/>
-    <geometry>
-      <mesh filename="file://$(find bebopv2_description)/meshes/foot_right_1.stl" scale="0.001 0.001 0.001"/>
-    </geometry>
-  </collision>
-</link>
 <link name="hip_flexion_right_1">
   <inertial>
@@ -126,5 +86,5 @@
 <link name="hip_flexion_left_1">
   <inertial>
-    <origin xyz="0.0013616527842525484 0.005166034468434444 -0.11306634650440041" rpy="0 0 0"/>
+    <origin xyz="0.0013616527842525501 0.005166034468434444 -0.11306634650440041" rpy="0 0 0"/>
     <mass value="1.1494341700004236"/>
     <inertia ixx="0.004841" iyy="0.004393" izz="0.00166" ixy="8e-06" iyz="-0.000393" ixz="4e-05"/>
@@ -181,4 +141,44 @@
     <geometry>
       <mesh filename="file://$(find bebopv2_description)/meshes/hip_abduction_left_1.stl" scale="0.001 0.001 0.001"/>
+    </geometry>
+  </collision>
+</link>
+<link name="foot_right_1">
+  <inertial>
+    <origin xyz="0.011485686877247665 0.022215465357853237 -0.023509071789787894" rpy="0 0 0"/>
+    <mass value="0.8000056692711454"/>
+    <inertia ixx="0.001043" iyy="0.002541" izz="0.002558" ixy="-0.0" iyz="0.0" ixz="0.00016"/>
+  </inertial>
+  <visual>
+    <origin xyz="-0.059094 0.178 0.674495" rpy="0 0 0"/>
+    <geometry>
+      <mesh filename="file://$(find bebopv2_description)/meshes/foot_right_1.stl" scale="0.001 0.001 0.001"/>
+    </geometry>
+    <material name="silver"/>
+  </visual>
+  <collision>
+    <origin xyz="-0.059094 0.178 0.674495" rpy="0 0 0"/>
+    <geometry>
+      <mesh filename="file://$(find bebopv2_description)/meshes/foot_right_1.stl" scale="0.001 0.001 0.001"/>
+    </geometry>
+  </collision>
+</link>
+<link name="foot_left_1">
+  <inertial>
+    <origin xyz="0.011473956574195115 -0.025038911721186607 -0.023484348928246468" rpy="0 0 0"/>
+    <mass value="0.7999816122276703"/>
+    <inertia ixx="0.001044" iyy="0.002539" izz="0.002557" ixy="7e-06" iyz="-1.4e-05" ixz="0.00016"/>
+  </inertial>
+  <visual>
+    <origin xyz="-0.063265 -0.1782 0.674402" rpy="0 0 0"/>
+    <geometry>
+      <mesh filename="file://$(find bebopv2_description)/meshes/foot_left_1.stl" scale="0.001 0.001 0.001"/>
+    </geometry>
+    <material name="silver"/>
+  </visual>
+  <collision>
+    <origin xyz="-0.063265 -0.1782 0.674402" rpy="0 0 0"/>
+    <geometry>
+      <mesh filename="file://$(find bebopv2_description)/meshes/foot_left_1.stl" scale="0.001 0.001 0.001"/>
     </geometry>
   </collision>
@@ -198,4 +198,39 @@
   <limit upper="0.785398" lower="-1.570796" effort="100" velocity="100"/>
 </joint>
+<joint name="hip_flexion_right_joint" type="revolute">
+  <origin xyz="-0.003527 -0.1503 0.013" rpy="0 0 0"/>
+  <parent link="base_link"/>
+  <child link="hip_flexion_right_1"/>
+  <axis xyz="-0.0 -1.0 -0.0"/>
+  <limit upper="0.785398" lower="-0.785398" effort="100" velocity="100"/>
+</joint>
+<joint name="hip_flexion_left_joint" type="revolute">
+  <origin xyz="-0.003789 0.1505 0.013132" rpy="0 0 0"/>
+  <parent link="base_link"/>
+  <child link="hip_flexion_left_1"/>
+  <axis xyz="0.0 1.0 -0.0"/>
+  <limit upper="0.785398" lower="-0.785398" effort="100" velocity="100"/>
+</joint>
+<joint name="hip_abduction_right_joint" type="revolute">
+  <origin xyz="0.02955 0.0 -0.14" rpy="0 0 0"/>
+  <parent link="hip_flexion_right_1"/>
+  <child link="hip_abduction_right_1"/>
+  <axis xyz="1.0 0.0 0.0"/>
+  <limit upper="0.174533" lower="-0.349066" effort="100" velocity="100"/>
+</joint>
+<joint name="hip_abduction_left_joint" type="revolute">
+  <origin xyz="0.02955 0.0 -0.14" rpy="0 0 0"/>
+  <parent link="hip_flexion_left_1"/>
+  <child link="hip_abduction_left_1"/>
+  <axis xyz="1.0 -0.0 0.0"/>
+  <limit upper="0.349066" lower="-0.174533" effort="100" velocity="100"/>
+</joint>
+<joint name="foot_right_joint" type="revolute">
+  <origin xyz="-0.004429 0.0 -0.253461" rpy="0 0 0"/>
+  <parent link="knee_flexion_right_1"/>
+  <child link="foot_right_1"/>
+  <axis xyz="-0.0 -1.0 -0.0"/>
+  <limit upper="0.523599" lower="-0.523599" effort="100" velocity="100"/>
+</joint>
 <joint name="foot_left_joint" type="revolute">
   <origin xyz="4e-06 0.0 -0.2535" rpy="0 0 0"/>
@@ -205,38 +240,3 @@
   <limit upper="0.523599" lower="-0.523599" effort="100" velocity="100"/>
 </joint>
-<joint name="foot_right_joint" type="revolute">
-  <origin xyz="-0.004429 0.0 -0.253461" rpy="0 0 0"/>
-  <parent link="knee_flexion_right_1"/>
-  <child link="foot_right_1"/>
-  <axis xyz="-0.0 -1.0 -0.0"/>
-  <limit upper="0.523599" lower="-0.523599" effort="100" velocity="100"/>
-</joint>
-<joint name="hip_flexion_right_joint" type="revolute">
-  <origin xyz="-0.003527 -0.1503 0.013" rpy="0 0 0"/>
-  <parent link="base_link"/>
-  <child link="hip_flexion_right_1"/>
-  <axis xyz="-0.0 -1.0 -0.0"/>
-  <limit upper="0.785398" lower="-0.785398" effort="100" velocity="100"/>
-</joint>
-<joint name="hip_flexion_left_joint" type="revolute">
-  <origin xyz="-0.003789 0.1505 0.013132" rpy="0 0 0"/>
-  <parent link="base_link"/>
-  <child link="hip_flexion_left_1"/>
-  <axis xyz="0.0 1.0 -0.0"/>
-  <limit upper="0.785398" lower="-0.785398" effort="100" velocity="100"/>
-</joint>
-<joint name="hip_abduction_right_joint" type="revolute">
-  <origin xyz="0.02955 0.0 -0.14" rpy="0 0 0"/>
-  <parent link="hip_flexion_right_1"/>
-  <child link="hip_abduction_right_1"/>
-  <axis xyz="1.0 0.0 0.0"/>
-  <limit upper="0.174533" lower="-0.349066" effort="100" velocity="100"/>
-</joint>
-<joint name="hip_abduction_left_joint" type="revolute">
-  <origin xyz="0.02955 0.0 -0.14" rpy="0 0 0"/>
-  <parent link="hip_flexion_left_1"/>
-  <child link="hip_abduction_left_1"/>
-  <axis xyz="1.0 -0.0 0.0"/>
-  <limit upper="0.349066" lower="-0.174533" effort="100" velocity="100"/>
-</joint>
 </robot>
