Commit message: added more foxglove tooling

File: ros2/src/bebopv2_description/urdf/bebopv2.urdf (robot description, URDF)
Before this commit: robot bebopv2, 9 links, 8 joints
Links:
- link base_link: geometry collision mesh filename=package://bebopv2_description/meshes/base_link.stl scale=0.001 0.001 0.001; visual mesh filename=package://bebopv2_description/meshes/base_link.stl scale=0.001 0.001 0.001
- link foot_left_1: geometry collision mesh filename=package://bebopv2_description/meshes/foot_left_1.stl scale=0.001 0.001 0.001; visual mesh filename=package://bebopv2_description/meshes/foot_left_1.stl scale=0.001 0.001 0.001
- link foot_right_1: geometry collision mesh filename=package://bebopv2_description/meshes/foot_right_1.stl scale=0.001 0.001 0.001; visual mesh filename=package://bebopv2_description/meshes/foot_right_1.stl scale=0.001 0.001 0.001
- link hip_abduction_left_1: geometry collision mesh filename=package://bebopv2_description/meshes/hip_abduction_left_1.s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 scale=0.001 0.001 0.001; visual mesh filename=package://bebopv2_description/meshes/hip_abduction_left_1.s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 scale=0.001 0.001 0.001
- link hip_abduction_right_1: geometry collision mesh filename=package://bebopv2_description/meshes/hip_abduction_right_1.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 scale=0.001 0.001 0.001; visual mesh filename=package://bebopv2_description/meshes/hip_abduction_right_1.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 scale=0.001 0.001 0.001
- link hip_flexion_left_1: geometry collision mesh filename=package://bebopv2_description/meshes/hip_flexion_left_1.stl scale=0.001 0.001 0.001; visual mesh filename=package://bebopv2_description/meshes/hip_flexion_left_1.stl scale=0.001 0.001 0.001
- link hip_flexion_right_1: geometry collision mesh filename=package://bebopv2_description/meshes/hip_flexion_right_1.stl scale=0.001 0.001 0.001; visual mesh filename=package://bebopv2_description/meshes/hip_flexion_right_1.stl scale=0.001 0.001 0.001
- link knee_flexion_left_1: geometry collision mesh filename=package://bebopv2_description/meshes/knee_flexion_left_1.stl scale=0.001 0.001 0.001; visual mesh filename=package://bebopv2_description/meshes/knee_flexion_left_1.stl scale=0.001 0.001 0.001
- link knee_flexion_right_1: geometry collision mesh filename=package://bebopv2_description/meshes/knee_flexion_right_1.s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 scale=0.001 0.001 0.001; visual mesh filename=package://bebopv2_description/meshes/knee_flexion_right_1.s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 scale=0.001 0.001 0.001
